Commit message: Husky with custom top plate

File: auto_landing/urdf/decorations.urdf.xacro (robot description, xacro)
@@ -152,5 +152,5 @@
             <origin xyz="0 0 0" rpy="0 0 0" />
             <geometry>
-              <mesh filename="package://husky_description/meshes/top_plate.dae" />
+              <mesh filename="package://auto_landing/meshes/custom_top_plate.dae" />
             </geometry>
           </visual>
@@ -158,5 +158,5 @@
             <origin xyz="0 0 0" rpy="0 0 0"/>
             <geometry>
-              <mesh filename="package://husky_description/meshes/top_plate.stl" />
+              <mesh filename="package://auto_landing/meshes/custom_top_plate.stl" />
             </geometry>
           </collision>
